File: ESP8266 w altanie/ESP8266 w altanie.sch (KiCad schematic (older format))
At the start: 29 parts, among them IC1 MCP23017-E_SP, Q1 2N2222A, Q2 2N2222A, Q3 2N2222A, Q4 2N2222A, Q5 2N2222A, Q6 2N2222A, Q7 2N2222A, Q8 2N2222A, SW1 SW_Push, SW2 SW_Push, SW3 SW_Push, SW4 SW_Push, U1 230VAC to 5VDC, U2 5vto3.3v, U3 ESP-07, U4 8x_Arduino_Relay_SSR

Commit message: Cleaning
Parts:
- U4: symbol Arduino_Relay:8x_Arduino_Relay_SSR -> ESP8266-w-altanie-rescue:8x_Arduino_Relay_SSR-Arduino_Relay
Changed lines of the file:
@@
 Connection ~ 7450 6150
 $Comp
-L Arduino_Relay:8x_Arduino_Relay_SSR U4
+L ESP8266-w-altanie-rescue:8x_Arduino_Relay_SSR-Arduino_Relay U4
 U 1 1 5F952CC1
 P 8850 3150
