File: Strych/Blinds.sch (KiCad schematic (older format))
At the start: 29 parts

Commit message: Strych board v0.1
Parts:
- added R65: 120, Resistor_THT:R_Axial_DIN0204_L3.6mm_D1.6mm_P7.62mm_Horizontal, symbol Device:R
- IC1, IC2: renamed from IC?; footprint DIP254P762X508-16 -> Package_DIP:DIP-16_W7.62mm
- Q1, Q2, Q3, Q4, Q5, Q6, Q7, Q8: renamed from Q?; footprint Package_TO_SOT_THT:TO-92_Inline -> Package_TO_SOT_THT:TO-92
- R1, R10, R11, R12, R13, R14, R15, R16, R2, R3, R4, R5, R6, R7, R8, R9: renamed from R?; footprint (none) -> Resistor_THT:R_Axial_DIN0204_L3.6mm_D1.6mm_P7.62mm_Horizontal
- U2: renamed from U?; footprint (none) -> Arduino Relay:MAX485
- U3: renamed from U?; footprint (none) -> Connector_PinSocket_2.54mm:PinSocket_1x10_P2.54mm_Vertical
- gave numbers to parts that had none: 1
Connections:
- net RS_A: now also R65.2
- net RS_B: now also R65.1
